File: mega-wifi.kicad_pcb (KiCad board)
At the start: 2 copper layers, 83.8 x 51 mm, 51 parts, among them P1 NP, P2 MD-CART-FINGERS, Q1 2N7002, U1 SC16C550BIB48, U2 S29GL032N, U3 ESP-12E, U4 AZ1117CH-3.3, U5 74LVC1G08GW, U6 74LVC162245, U7 74LVC245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

Commit message: Update to KiCad 7
Other:
- net class Default removed
- net class POWER removed
