File: mega-wifi.kicad_pcb (KiCad board)
At the start: 2 copper layers, 83.8 x 51 mm, 55 parts, among them P1 MD-CART-FINGERS, P2 USB_C_Receptacle_USB2.0_16P, Q1 2N7002, Q2 2N7002, U1 74LVC08, U2 AMS1117-3.3, U3 74LVC16245, U4 74LVC245, U5 74LVC16245, U6 S29GL064N, U7 SC16C550BIBS, U8 ESP32-C3-WROOM-02, Y1 24 MHz

Commit message: Rev.C: replace SC16C550BIBS with TI TL16C550DRHB
The NXP SC16C550BIBS is out of stock everywhere. The TI TL16C550D in the
RHB (5x5 VQFN-32) package is pin-for-pin compatible and register
compatible (auto RTS/CTS via MCR AFE), so the existing driver works.

- U7: TL16C550DRHB (LCSC C2653239), Texas RHB0032E footprint (EP 3.45 mm,
  perimeter pads unchanged); pin names updated to TI naming.
- Y1: 20 MHz crystal (TXC 7E20000E12UCG, C252261, 12 pF load). TI rates
  the RHB package to 20 MHz at 3.3 V, so the UART link runs at
  1.25 Mbaud (divisor 1). SGDK 16c550.h and mw-fw-rtos LSD_UART_BR must
  be set to match; existing ROMs/firmware at 1.5 Mbaud will not work.
- R18: 1 MOhm oscillator bias resistor across XIN/XOUT (C26083); the TI
  oscillator has no internal Rp, unlike the NXP part.
- RI (pin 27) tied to VCC; the TI part has no internal modem-input
  pull-ups.
- XIN/XOUT nets are now labelled (/WiFi/XIN, /WiFi/XOUT).
- Zones refilled.
- Revision bumped to Rev.C (title blocks and silkscreen), credits
  doragasu 2024, jfryman 2026.

Files remain in KiCad 8 format.

Co-Authored-By: Claude Opus 5.5 <noreply@anthropic.com>
Parts:
- added R18: 1M, Resistor_SMD:R_0402_1005Metric, F.Cu at (155.2, 86.3)
- U7: value SC16C550BIBS -> TL16C550DRHB; footprint Package_DFN_QFN:HVQFN-32-1EP_5x5mm_P0.5mm_EP3.1x3.1mm -> Package_DFN_QFN:Texas_RHB0032E_VQFN-32-1EP_5x5mm_P0.5mm_EP3.45x3.45mm
- Y1: value 24 MHz -> 20 MHz
Connections:
- net Net-(U7-XTAL1) renamed /WiFi/XIN
- net Net-(U7-XTAL2) renamed /WiFi/XOUT
- U7 pad 27: unconnected-(U7-~{RI}-Pad27) -> VCC
Routing:
- net VCC: track 108.1 -> 109.5 mm
Other:
- board text added: "MegaWiFi Rev.C doragasu 2024 jfryman 2026"
- board text added: "MegaWiFi Rev.C, doragasu 2024, jfryman 2026"
- board text removed: "MegaWiFi Rev.B doragasu 2024"
- board text removed: "MegaWiFi Rev.B, doragasu 2024"
