File: mega-wifi.kicad_sch (KiCad schematic)
At the start: 23 parts, among them P1 MD-CART-FINGERS, U1 74LVC08, U2 AMS1117-3.3, U3 74LVC16245, U4 74LVC245, U5 74LVC16245

Commit message: Rev.C: replace SC16C550BIBS with TI TL16C550DRHB
The NXP SC16C550BIBS is out of stock everywhere. The TI TL16C550D in the
RHB (5x5 VQFN-32) package is pin-for-pin compatible and register
compatible (auto RTS/CTS via MCR AFE), so the existing driver works.

- U7: TL16C550DRHB (LCSC C2653239), Texas RHB0032E footprint (EP 3.45 mm,
  perimeter pads unchanged); pin names updated to TI naming.
- Y1: 20 MHz crystal (TXC 7E20000E12UCG, C252261, 12 pF load). TI rates
  the RHB package to 20 MHz at 3.3 V, so the UART link runs at
  1.25 Mbaud (divisor 1). SGDK 16c550.h and mw-fw-rtos LSD_UART_BR must
  be set to match; existing ROMs/firmware at 1.5 Mbaud will not work.
- R18: 1 MOhm oscillator bias resistor across XIN/XOUT (C26083); the TI
  oscillator has no internal Rp, unlike the NXP part.
- RI (pin 27) tied to VCC; the TI part has no internal modem-input
  pull-ups.
- XIN/XOUT nets are now labelled (/WiFi/XIN, /WiFi/XOUT).
- Zones refilled.
- Revision bumped to Rev.C (title blocks and silkscreen), credits
  doragasu 2024, jfryman 2026.

Files remain in KiCad 8 format.

Co-Authored-By: Claude Opus 5.5 <noreply@anthropic.com>
Other:
- company: doragasu -> doragasu, jfryman
Changed lines of the file:
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@@
 	(title_block
 		(title "MegaWiFi")
-		(date "2024-10-07")
-		(rev "B")
-		(company "doragasu")
+		(date "2026-10-06")
+		(rev "C")
+		(company "doragasu, jfryman")
 		(comment 1 "License: CERN OHL 1.2")
+		(comment 2 "Rev.C: TL16C550D UART, 20 MHz clock")
 		(comment 4 "CART AND TRANSCEIVERS")
 	)
